File: hardware/kicad-project/Untitled.kicad_pcb (KiCad board)
At the start: 2 copper layers, 110 x 70 mm, 75 parts, among them CN2 ST-0322D00-071-1A2H, J8 Conn_01x50, Q1 DMG2301L-7, Q2 DMG2301L-7, Q3 DMG2301L-7, SW1 TS-1187A-B-A-B, SW10 TS-1135-C, SW2 TS-1187A-B-A-B, SW4 K2-1109SP-C4SA, SW5 K2-1109SP-C4SA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

Commit message: reset schemtics to rev1
Connections:
- CN2 pad 1: Net-(U6-OUTN) -> GND
- H2 pad 1: Net-(U6-OUTN) -> GND
- U6 pad 10: Net-(U6-OUTN) -> GND
Routing:
- net Net-(U6-OUTN): track 99.1 -> 0.00 mm, vias 2 -> 0
- net GND: track 62.0 -> 65.0 mm
Changed lines of the file:
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@@
   (net 104 "unconnected-(CN2-Pad7)")
   (net 105 "unconnected-(Card1-PadCD)")
-  (net 106 "Net-(U6-OUTN)")
   (footprint "Resistor_SMD:R_0603_1608Metric" (layer "F.Cu")
     (at 97.175 98)
@@
       (stroke (width 0.06) (type solid)) (fill none) (layer "F.Fab"))
     (pad "1" smd rect (at -1 -2.85 270) (size 1 3.5) (layers "F.Cu" "F.Paste" "F.Mask")
-      (net 106 "Net-(U6-OUTN)") (pinfunction "1") (pintype "unspecified"))
+      (net 3 "GND") (pinfunction "1") (pintype "unspecified"))
     (pad "2" smd rect (at 1 -2.85 270) (size 1 3.5) (layers "F.Cu" "F.Paste" "F.Mask")
       (net 37 "Net-(CN2-Pad5)") (pinfunction "2") (pintype "unspecified"))
@@
     (pad "" thru_hole circle (at 2.65 0.26) (size 1.5 1.5) (drill 1.5) (layers "*.Cu" "*.Mask"))
     (pad "1" thru_hole oval (at -4.65 3) (size 2 1) (drill oval 1.399997 0.599999) (layers "*.Cu" "*.Mask")
-      (net 106 "Net-(U6-OUTN)") (pinfunction "1") (pintype "unspecified"))
+      (net 3 "GND") (pinfunction "1") (pintype "unspecified"))
     (pad "2" thru_hole oval (at -4.65 -2.13) (size 2 1) (drill oval 1.399997 0.599999) (layers "*.Cu" "*.Mask")
       (net 36 "Net-(U6-OUTP)") (pinfunction "2") (pintype "unspecified"))
@@
       (net 36 "Net-(U6-OUTP)") (pinfunction "OUTP") (pintype "unspecified"))
     (pad "10" smd rect (at 0.25 -1.5 90) (size 0.25 0.6) (layers "F.Cu" "F.Paste" "F.Mask")
-      (net 106 "Net-(U6-OUTN)") (pinfunction "OUTN") (pintype "unspecified"))
+      (net 3 "GND") (pinfunction "OUTN") (pintype "unspecified"))
     (pad "11" smd rect (at -0.25 -1.5 90) (size 0.25 0.6) (layers "F.Cu" "F.Paste" "F.Mask")
       (net 3 "GND") (pinfunction "GND") (pintype "unspecified"))
@@
   (segment (start 118.297576 104.312356) (end 118.297576 106.212356) (width 0.25) (layer "F.Cu") (net 3))
   (segment (start 122 106.312356) (end 122 106.484932) (width 0.25) (layer "F.Cu") (net 3))
-  (segment (start 107.409682 119.75) (end 108.659682 119.75) (width 0.25) (layer "F.Cu") (net 3))
   (segment (start 152.276163 70.563886) (end 153.925978 68.914071) (width 0.25) (layer "F.Cu") (net 3))
   (segment (start 118.297576 106.212356) (end 118.397576 106.312356) (width 0.25) (layer "F.Cu") (net 3))
@@
   (segment (start 122 106.312356) (end 122.172576 106.312356) (width 0.25) (layer "F.Cu") (net 3))
   (segment (start 121.372576 107.112356) (end 119.197576 107.112356) (width 0.25) (layer "F.Cu") (net 3))
+  (segment (start 107.409682 119.25) (end 106.05 119.25) (width 0.25) (layer "F.Cu") (net 3))
   (segment (start 95 98.623393) (end 95.267824 98.891217) (width 0.3) (layer "F.Cu") (net 3))
   (segment (start 119.197576 107.112356) (end 118.397576 106.312356) (width 0.25) (layer "F.Cu") (net 3))
   (segment (start 151.226163 91.563886) (end 151.226163 92.563886) (width 0.25) (layer "F.Cu") (net 3))
   (segment (start 151.226163 73.063886) (end 151.226163 73.563886) (width 0.25) (layer "F.Cu") (net 3))
+  (segment (start 107.409682 119.75) (end 106.55 119.75) (width 0.25) (layer "F.Cu") (net 3))
   (segment (start 151.226163 91.563886) (end 152.436114 91.563886) (width 0.25) (layer "F.Cu") (net 3))
   (segment (start 97.108783 98.891217) (end 98 98) (width 0.3) (layer "F.Cu") (net 3))
@@
   (segment (start 98.594549 110.022072) (end 99.144549 109.472072) (width 0.25) (layer "F.Cu") (net 3))
   (segment (start 95 95.775) (end 95 98.623393) (width 0.3) (layer "F.Cu") (net 3))
+  (segment (start 106.55 119.75) (end 106.05 119.25) (width 0.25) (layer "F.Cu") (net 3))
   (segment (start 95.275 95.5) (end 95 95.775) (width 0.3) (layer "F.Cu") (net 3))
   (segment (start 114.622416 118.597111) (end 116.328795 118.597111) (width 0.25) (layer "F.Cu") (net 3))
   (segment (start 99.144549 103.072072) (end 100.496915 103.072072) (width 0.25) (layer "F.Cu") (net 3))
   (segment (start 109.159682 119.25) (end 108.909682 119.5) (width 0.25) (layer "F.Cu") (net 3))
+  (segment (start 107.409682 119.25) (end 108.659682 119.25) (width 0.25) (layer "F.Cu") (net 3))
   (segment (start 151.226163 89.063886) (end 152.276163 89.063886) (width 0.25) (layer "F.Cu") (net 3))
+  (segment (start 106 119.2) (end 106.05 119.25) (width 0.25) (layer "F.Cu") (net 3))
   (via (at 107 75) (size 0.8) (drill 0.4) (layers "F.Cu" "B.Cu") (free) (net 3))
   (via (at 104 75) (size 0.8) (drill 0.4) (layers "F.Cu" "B.Cu") (free) (net 3))
@@
   (segment (start 135 75) (end 159.380988 75) (width 0.25) (layer "B.Cu") (net 92))
   (segment (start 170.16634 73.83366) (end 171 73) (width 0.25) (layer "B.Cu") (net 92))
-  (segment (start 164.81304 100) (end 169.386717 104.573677) (width 0.25) (layer "F.Cu") (net 106))
-  (segment (start 99.257818 121.404078) (end 100.85374 123) (width 0.25) (layer "F.Cu") (net 106))
-  (segment (start 138 100) (end 164.81304 100) (width 0.25) (layer "F.Cu") (net 106))
-  (segment (start 137 99) (end 138 100) (width 0.25) (layer "F.Cu") (net 106))
-  (segment (start 105.415318 119.415318) (end 106.784682 119.415318) (width 0.25) (layer "F.Cu") (net 106))
-  (segment (start 106.95 119.25) (end 107.409682 119.25) (width 0.25) (layer "F.Cu") (net 106))
-  (segment (start 169.386717 104.573677) (end 169.386717 105.323677) (width 0.25) (layer "F.Cu") (net 106))
-  (segment (start 106.784682 119.415318) (end 106.95 119.25) (width 0.25) (layer "F.Cu") (net 106))
-  (segment (start 94.824544 121.404078) (end 99.257818 121.404078) (width 0.25) (layer "F.Cu") (net 106))
-  (segment (start 104.195348 123) (end 105.449544 121.745804) (width 0.25) (layer "F.Cu") (net 106))
-  (segment (start 105.449544 119.449544) (end 105 119) (width 0.25) (layer "F.Cu") (net 106))
-  (segment (start 100.85374 123) (end 104.195348 123) (width 0.25) (layer "F.Cu") (net 106))
-  (segment (start 105 119) (end 105.415318 119.415318) (width 0.25) (layer "F.Cu") (net 106))
-  (segment (start 105.449544 121.745804) (end 105.449544 119.449544) (width 0.25) (layer "F.Cu") (net 106))
-  (via (at 105 119) (size 0.8) (drill 0.4) (layers "F.Cu" "B.Cu") (net 106))
-  (via (at 137 99) (size 0.8) (drill 0.4) (layers "F.Cu" "B.Cu") (net 106))
-  (segment (start 105 119) (end 105 119.862734) (width 0.25) (layer "B.Cu") (net 106))
-  (segment (start 116.732413 123) (end 126.475 113.257413) (width 0.25) (layer "B.Cu") (net 106))
-  (segment (start 105 119.862734) (end 108.137266 123) (width 0.25) (layer "B.Cu") (net 106))
-  (segment (start 126.475 109.525) (end 137 99) (width 0.25) (layer "B.Cu") (net 106))
-  (segment (start 126.475 113.257413) (end 126.475 109.525) (width 0.25) (layer "B.Cu") (net 106))
-  (segment (start 108.137266 123) (end 116.732413 123) (width 0.25) (layer "B.Cu") (net 106))
   (zone (net 3) (net_name "GND") (layer "F.Cu") (hatch edge 0.5)
     (connect_pads (clearance 0.5))
