File: hardware/kicad-project/random.kicad_sch (KiCad schematic)
At the start: 33 parts, among them J7 Conn_01x50, Q3 DMG2301L-7, SW10 TS-1135-C, SW4 K2-1109SP-C4SA, SW5 K2-1109SP-C4SA, SW6 K2-1109SP-C4SA, SW7 K2-1109SP-C4SA, SW8 TS-1135-C, SW9 TS-1135-C

Commit message: wip
Connections:
- net CONTROLLED_3.3V is gone; now on net +3.3V: C10.2, C12.2, C12.2, C13.1, C9.2, Card1.4 (VDD), J7.40 (Pin_40), J7.41 (Pin_41), J7.42 (Pin_41), R19.2, R21.2, R22.2, R23.2, R24.2, R25.2
Changed lines of the file:
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@@
   (junction (at 57.15 149.86) (diameter 0) (color 0 0 0 0)
   )
+  (junction (at 31.75 143.51) (diameter 0) (color 0 0 0 0)
+  )
   (junction (at 96.52 76.2) (diameter 0) (color 0 0 0 0)
   )
@@
   )
   (junction (at 96.52 127) (diameter 0) (color 0 0 0 0)
-  )
-  (junction (at 31.75 143.51) (diameter 0) (color 0 0 0 0)
   )
   (junction (at 165.1 110.49) (diameter 0) (color 0 0 0 0)
@@
     (stroke (width 0) (type default))
   )
-  (wire (pts (xy 223.52 21.59) (xy 223.52 27.94))
-    (stroke (width 0) (type default))
-  )
-  (wire (pts (xy 214.63 21.59) (xy 223.52 21.59))
+  (wire (pts (xy 223.52 25.4) (xy 223.52 27.94))
     (stroke (width 0) (type default))
   )
@@
   )
   (wire (pts (xy 223.52 50.8) (xy 233.68 50.8))
-    (stroke (width 0) (type default))
-  )
-  (wire (pts (xy 29.21 143.51) (xy 31.75 143.51))
     (stroke (width 0) (type default))
   )
@@
     (effects (font (size 1.27 1.27)) (justify right))
     (property "Intersheetrefs" "${INTERSHEET_REFS}" (at 127.1596 53.34 0)
-      (effects (font (size 1.27 1.27)) (justify right) hide)
-    )
-  )
-  (global_label "CONTROLLED_3.3V" (shape input) (at 29.21 143.51 180) (fields_autoplaced)
-    (effects (font (size 1.27 1.27)) (justify right))
-    (property "Intersheetrefs" "${INTERSHEET_REFS}" (at 9.1705 143.51 0)
-      (effects (font (size 1.27 1.27)) (justify right) hide)
-    )
-  )
-  (global_label "CONTROLLED_3.3V" (shape input) (at 214.63 21.59 180) (fields_autoplaced)
-    (effects (font (size 1.27 1.27)) (justify right))
-    (property "Intersheetrefs" "${INTERSHEET_REFS}" (at 194.5905 21.59 0)
       (effects (font (size 1.27 1.27)) (justify right) hide)
     )
@@
     )
   )
+  (symbol (lib_id "power:+3.3V") (at 223.52 25.4 0) (unit 1)
+    (in_bom yes) (on_board yes) (dnp no) (fields_autoplaced)
+    (property "Reference" "#PWR030" (at 223.52 29.21 0)
+      (effects (font (size 1.27 1.27)) hide)
+    )
+    (property "Value" "+3.3V" (at 223.52 20.32 0)
+      (effects (font (size 1.27 1.27)))
+    )
+    (property "Footprint" "" (at 223.52 25.4 0)
+      (effects (font (size 1.27 1.27)) hide)
+    )
+    (property "Datasheet" "" (at 223.52 25.4 0)
+      (effects (font (size 1.27 1.27)) hide)
+    )
+    (pin "1")
+    (instances
+      (project "Untitled"
+        (path "/0de5ae84-7f75-4a5a-83a1-35d27fd1d8d2"
+          (reference "#PWR030") (unit 1)
+        )
+        (path "/0de5ae84-7f75-4a5a-83a1-35d27fd1d8d2/7a3aed0a-25fa-4aa7-ba6a-02a8683cfb94"
+          (reference "#PWR043") (unit 1)
+        )
+      )
+    )
+  )
   (symbol (lib_id "power:GND") (at 74.93 60.96 0) (unit 1)
     (in_bom yes) (on_board yes) (dnp no)
@@
         )
       )
+    )
+  )
+  (symbol (lib_id "power:+3.3V") (at 31.75 143.51 0) (unit 1)
+    (in_bom yes) (on_board yes) (dnp no) (fields_autoplaced)
+    (property "Reference" "#PWR030" (at 31.75 147.32 0)
+      (effects (font (size 1.27 1.27)) hide)
+    )
+    (property "Value" "+3.3V" (at 31.75 138.43 0)
+      (effects (font (size 1.27 1.27)))
+    )
+    (property "Footprint" "" (at 31.75 143.51 0)
+      (effects (font (size 1.27 1.27)) hide)
+    )
+    (property "Datasheet" "" (at 31.75 143.51 0)
+      (effects (font (size 1.27 1.27)) hide)
+    )
+    (pin "1")
+    (instances
+      (project "Untitled"
+        (path "/0de5ae84-7f75-4a5a-83a1-35d27fd1d8d2"
+          (reference "#PWR030") (unit 1)
+        )
+        (path "/0de5ae84-7f75-4a5a-83a1-35d27fd1d8d2/7a3aed0a-25fa-4aa7-ba6a-02a8683cfb94"
+          (reference "#PWR042") (unit 1)
+        )
+      )

Commit message: New side buttons
Parts:
- removed SW10, SW8, SW9: TS-1135-C, easyeda2kicad:SW-SMD_YIYUAN_YTS-B017-2H, symbol easyedaToKicad:TS-1135-C
- added U4, U5, U7: GT-TC054C-H035-L1W, easyeda2kicad:KEY-SMD_4P-L7.8-W2.8-P4.20-EH, symbol easyedaToKicad:GT-TC054C-H035-L1W
Connections:
- net BTN_5: now also U4.1
- net BTN_6: now also U5.1
- net BTN_7: now also U7.1
- net GND: now also U4.2, U5.2, U7.2

Commit message: wip
Parts:
- renumbered SW4 to SW1, SW5 to SW2, SW6 to SW3, SW7 to SW4, U4 to SW5, U5 to SW6, U7 to SW7
Changed lines of the file:
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@@
   (junction (at 96.52 78.74) (diameter 0) (color 0 0 0 0)
   )
+  (junction (at 96.52 172.72) (diameter 0) (color 0 0 0 0)
+  )
+  (junction (at 208.28 27.94) (diameter 0) (color 0 0 0 0)
+  )
+  (junction (at 165.1 96.52) (diameter 0) (color 0 0 0 0)
+  )
+  (junction (at 96.52 116.84) (diameter 0) (color 0 0 0 0)
+  )
+  (junction (at 165.1 64.77) (diameter 0) (color 0 0 0 0)
+  )
+  (junction (at 254 33.02) (diameter 0) (color 0 0 0 0)
+  )
+  (junction (at 165.1 81.28) (diameter 0) (color 0 0 0 0)
+  )
+  (junction (at 207.01 91.44) (diameter 0) (color 0 0 0 0)
+  )
+  (junction (at 88.9 68.58) (diameter 0) (color 0 0 0 0)
+  )
+  (junction (at 212.09 40.64) (diameter 0) (color 0 0 0 0)
+  )
+  (junction (at 201.93 91.44) (diameter 0) (color 0 0 0 0)
+  )
+  (junction (at 200.66 27.94) (diameter 0) (color 0 0 0 0)
+  )
+  (junction (at 96.52 121.92) (diameter 0) (color 0 0 0 0)
+  )
+  (junction (at 57.15 147.32) (diameter 0) (color 0 0 0 0)
+  )
+  (junction (at 96.52 91.44) (diameter 0) (color 0 0 0 0)
+  )
+  (junction (at 96.52 124.46) (diameter 0) (color 0 0 0 0)
+  )
+  (junction (at 96.52 96.52) (diameter 0) (color 0 0 0 0)
+  )
+  (junction (at 57.15 152.4) (diameter 0) (color 0 0 0 0)
+  )
   (junction (at 60.96 68.58) (diameter 0) (color 0 0 0 0)
-  )
-  (junction (at 96.52 172.72) (diameter 0) (color 0 0 0 0)
-  )
-  (junction (at 208.28 27.94) (diameter 0) (color 0 0 0 0)
-  )
-  (junction (at 165.1 96.52) (diameter 0) (color 0 0 0 0)
-  )
-  (junction (at 96.52 116.84) (diameter 0) (color 0 0 0 0)
-  )
-  (junction (at 165.1 64.77) (diameter 0) (color 0 0 0 0)
-  )
-  (junction (at 254 33.02) (diameter 0) (color 0 0 0 0)
-  )
-  (junction (at 165.1 81.28) (diameter 0) (color 0 0 0 0)
-  )
-  (junction (at 207.01 91.44) (diameter 0) (color 0 0 0 0)
-  )
-  (junction (at 88.9 68.58) (diameter 0) (color 0 0 0 0)
-  )
-  (junction (at 212.09 40.64) (diameter 0) (color 0 0 0 0)
-  )
-  (junction (at 201.93 91.44) (diameter 0) (color 0 0 0 0)
-  )
-  (junction (at 200.66 27.94) (diameter 0) (color 0 0 0 0)
-  )
-  (junction (at 96.52 121.92) (diameter 0) (color 0 0 0 0)
-  )
-  (junction (at 57.15 147.32) (diameter 0) (color 0 0 0 0)
-  )
-  (junction (at 96.52 91.44) (diameter 0) (color 0 0 0 0)
-  )
-  (junction (at 96.52 124.46) (diameter 0) (color 0 0 0 0)
-  )
-  (junction (at 96.52 96.52) (diameter 0) (color 0 0 0 0)
-  )
-  (junction (at 57.15 152.4) (diameter 0) (color 0 0 0 0)
   )
   (junction (at 223.52 27.94) (diameter 0) (color 0 0 0 0)
@@
     (stroke (width 0) (type default))
   )
+  (wire (pts (xy 215.9 38.1) (xy 233.68 38.1))
+    (stroke (width 0) (type default))
+  )
+  (wire (pts (xy 93.98 142.24) (xy 99.06 142.24))
+    (stroke (width 0) (type default))
+  )
+  (wire (pts (xy 165.1 53.34) (xy 165.1 64.77))
+    (stroke (width 0) (type default))
+  )
+  (wire (pts (xy 96.52 124.46) (xy 99.06 124.46))
+    (stroke (width 0) (type default))
+  )
+  (wire (pts (xy 57.15 152.4) (xy 57.15 149.86))
+    (stroke (width 0) (type default))
+  )
   (wire (pts (xy 60.96 68.58) (xy 60.96 71.12))
-    (stroke (width 0) (type default))
-  )
-  (wire (pts (xy 215.9 38.1) (xy 233.68 38.1))
-    (stroke (width 0) (type default))
-  )
-  (wire (pts (xy 93.98 142.24) (xy 99.06 142.24))
-    (stroke (width 0) (type default))
-  )
-  (wire (pts (xy 165.1 53.34) (xy 165.1 64.77))
-    (stroke (width 0) (type default))
-  )
-  (wire (pts (xy 96.52 124.46) (xy 99.06 124.46))
-    (stroke (width 0) (type default))
-  )
-  (wire (pts (xy 57.15 152.4) (xy 57.15 149.86))
     (stroke (width 0) (type default))
   )
@@
   (symbol (lib_id "easyedaToKicad:GT-TC054C-H035-L1W") (at 148.59 110.49 0) (unit 1)
     (in_bom yes) (on_board yes) (dnp no) (fields_autoplaced)
-    (property "Reference" "U7" (at 148.59 104.14 0)
+    (property "Reference" "SW7" (at 148.59 104.14 0)
       (effects (font (size 1.27 1.27)))
     )
@@
       (project "Untitled"
         (path "/0de5ae84-7f75-4a5a-83a1-35d27fd1d8d2/7a3aed0a-25fa-4aa7-ba6a-02a8683cfb94"
-          (reference "U7") (unit 1)
+          (reference "SW7") (unit 1)
         )
       )
@@
   (symbol (lib_id "easyedaToKicad:K2-1109SP-C4SA") (at 147.32 33.02 90) (unit 1)
     (in_bom yes) (on_board yes) (dnp no) (fields_autoplaced)
-    (property "Reference" "SW4" (at 151.13 31.75 90)
+    (property "Reference" "SW1" (at 151.13 31.75 90)
       (effects (font (size 1.27 1.27)) (justify right))
     )
@@
       (project "Untitled"
         (path "/0de5ae84-7f75-4a5a-83a1-35d27fd1d8d2/7a3aed0a-25fa-4aa7-ba6a-02a8683cfb94"
-          (reference "SW4") (unit 1)
+          (reference "SW1") (unit 1)
         )
       )
@@
   (symbol (lib_id "easyedaToKicad:K2-1109SP-C4SA") (at 147.32 45.72 90) (unit 1)
     (in_bom yes) (on_board yes) (dnp no) (fields_autoplaced)
-    (property "Reference" "SW5" (at 151.13 44.45 90)
+    (property "Reference" "SW2" (at 151.13 44.45 90)
       (effects (font (size 1.27 1.27)) (justify right))
     )
@@
       (project "Untitled"
         (path "/0de5ae84-7f75-4a5a-83a1-35d27fd1d8d2/7a3aed0a-25fa-4aa7-ba6a-02a8683cfb94"
-          (reference "SW5") (unit 1)
+          (reference "SW2") (unit 1)
         )
       )
@@
   (symbol (lib_id "easyedaToKicad:GT-TC054C-H035-L1W") (at 148.59 96.52 0) (unit 1)
     (in_bom yes) (on_board yes) (dnp no) (fields_autoplaced)
-    (property "Reference" "U5" (at 148.59 90.17 0)
+    (property "Reference" "SW6" (at 148.59 90.17 0)
       (effects (font (size 1.27 1.27)))
     )
@@
       (project "Untitled"
         (path "/0de5ae84-7f75-4a5a-83a1-35d27fd1d8d2/7a3aed0a-25fa-4aa7-ba6a-02a8683cfb94"
-          (reference "U5") (unit 1)
+          (reference "SW6") (unit 1)
         )
       )
@@
   (symbol (lib_id "easyedaToKicad:GT-TC054C-H035-L1W") (at 148.59 81.28 0) (unit 1)
     (in_bom yes) (on_board yes) (dnp no) (fields_autoplaced)
-    (property "Reference" "U4" (at 148.59 74.93 0)
+    (property "Reference" "SW5" (at 148.59 74.93 0)
       (effects (font (size 1.27 1.27)))
     )
@@
       (project "Untitled"
         (path "/0de5ae84-7f75-4a5a-83a1-35d27fd1d8d2/7a3aed0a-25fa-4aa7-ba6a-02a8683cfb94"
-          (reference "U4") (unit 1)
+          (reference "SW5") (unit 1)
         )
       )
@@
   (symbol (lib_id "easyedaToKicad:K2-1109SP-C4SA") (at 147.32 57.15 90) (unit 1)
     (in_bom yes) (on_board yes) (dnp no) (fields_autoplaced)
-    (property "Reference" "SW6" (at 151.13 55.88 90)
+    (property "Reference" "SW3" (at 151.13 55.88 90)
       (effects (font (size 1.27 1.27)) (justify right))
     )
@@
       (project "Untitled"
         (path "/0de5ae84-7f75-4a5a-83a1-35d27fd1d8d2/7a3aed0a-25fa-4aa7-ba6a-02a8683cfb94"
-          (reference "SW6") (unit 1)
+          (reference "SW3") (unit 1)
         )
       )
@@
   (symbol (lib_id "easyedaToKicad:K2-1109SP-C4SA") (at 147.32 68.58 90) (unit 1)
     (in_bom yes) (on_board yes) (dnp no) (fields_autoplaced)
-    (property "Reference" "SW7" (at 151.13 67.31 90)
+    (property "Reference" "SW4" (at 151.13 67.31 90)
       (effects (font (size 1.27 1.27)) (justify right))
     )
@@
       (project "Untitled"
         (path "/0de5ae84-7f75-4a5a-83a1-35d27fd1d8d2/7a3aed0a-25fa-4aa7-ba6a-02a8683cfb94"
-          (reference "SW7") (unit 1)
-        )
-      )
+          (reference "SW4") (unit 1)
+        )
+      )

Commit message: update
Parts:
- C13: footprint Capacitor_SMD:C_0603_1608Metric -> Capacitor_SMD:C_0805_2012Metric
- R10, R17, R19, R20, R21, R22, R23, R24, R25, R9: footprint Resistor_SMD:R_0603_1608Metric -> Resistor_SMD:R_0805_2012Metric
Changed lines of the file:
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@@
       (effects (font (size 1.27 1.27)))
     )
-    (property "Footprint" "Resistor_SMD:R_0603_1608Metric" (at 78.74 51.562 90)
+    (property "Footprint" "Resistor_SMD:R_0805_2012Metric" (at 78.74 51.562 90)
       (effects (font (size 1.27 1.27)) hide)
     )
@@
       (effects (font (size 1.27 1.27)))
     )
-    (property "Footprint" "Resistor_SMD:R_0603_1608Metric" (at 77.47 69.342 90)
+    (property "Footprint" "Resistor_SMD:R_0805_2012Metric" (at 77.47 69.342 90)
       (effects (font (size 1.27 1.27)) hide)
     )
@@
       (effects (font (size 1.27 1.27)) (justify right))
     )
-    (property "Footprint" "Resistor_SMD:R_0603_1608Metric" (at 210.058 31.75 90)
+    (property "Footprint" "Resistor_SMD:R_0805_2012Metric" (at 210.058 31.75 90)
       (effects (font (size 1.27 1.27)) hide)
     )
@@
       (effects (font (size 1.27 1.27)) (justify right))
     )
-    (property "Footprint" "Resistor_SMD:R_0603_1608Metric" (at 38.1 42.418 90)
+    (property "Footprint" "Resistor_SMD:R_0805_2012Metric" (at 38.1 42.418 90)
       (effects (font (size 1.27 1.27)) hide)
     )
@@
       (effects (font (size 1.27 1.27)))
     )
-    (property "Footprint" "Resistor_SMD:R_0603_1608Metric" (at 86.36 54.102 90)
+    (property "Footprint" "Resistor_SMD:R_0805_2012Metric" (at 86.36 54.102 90)
       (effects (font (size 1.27 1.27)) hide)
     )
@@
       (effects (font (size 1.27 1.27)) (justify right))
     )
-    (property "Footprint" "Capacitor_SMD:C_0603_1608Metric" (at 68.8848 166.37 0)
+    (property "Footprint" "Capacitor_SMD:C_0805_2012Metric" (at 68.8848 166.37 0)
       (effects (font (size 1.27 1.27)) hide)
     )
@@
       (effects (font (size 1.27 1.27)) (justify right))
     )
-    (property "Footprint" "Resistor_SMD:R_0603_1608Metric" (at 217.678 31.75 90)
+    (property "Footprint" "Resistor_SMD:R_0805_2012Metric" (at 217.678 31.75 90)
       (effects (font (size 1.27 1.27)) hide)
     )
@@
       (effects (font (size 1.27 1.27)) (justify right))
     )
-    (property "Footprint" "Resistor_SMD:R_0603_1608Metric" (at 198.628 31.75 90)
+    (property "Footprint" "Resistor_SMD:R_0805_2012Metric" (at 198.628 31.75 90)
       (effects (font (size 1.27 1.27)) hide)
     )
@@
       (effects (font (size 1.27 1.27)) (justify right))
     )
-    (property "Footprint" "Resistor_SMD:R_0603_1608Metric" (at 202.438 31.75 90)
+    (property "Footprint" "Resistor_SMD:R_0805_2012Metric" (at 202.438 31.75 90)
       (effects (font (size 1.27 1.27)) hide)
     )
@@
       (effects (font (size 1.27 1.27)) (justify right))
     )
-    (property "Footprint" "Resistor_SMD:R_0603_1608Metric" (at 213.868 31.75 90)
+    (property "Footprint" "Resistor_SMD:R_0805_2012Metric" (at 213.868 31.75 90)
       (effects (font (size 1.27 1.27)) hide)
     )
@@
       (effects (font (size 1.27 1.27)) (justify right))
     )
-    (property "Footprint" "Resistor_SMD:R_0603_1608Metric" (at 206.248 31.75 90)
+    (property "Footprint" "Resistor_SMD:R_0805_2012Metric" (at 206.248 31.75 90)
       (effects (font (size 1.27 1.27)) hide)
     )
@@
       (effects (font (size 1.27 1.27)))
     )
-    (property "Footprint" "Resistor_SMD:R_0603_1608Metric" (at 93.98 56.642 90)
+    (property "Footprint" "Resistor_SMD:R_0805_2012Metric" (at 93.98 56.642 90)
       (effects (font (size 1.27 1.27)) hide)
     )
@@
       (effects (font (size 1.27 1.27)) (justify right))
     )
-    (property "Footprint" "Resistor_SMD:R_0603_1608Metric" (at 44.958 34.29 90)
+    (property "Footprint" "Resistor_SMD:R_0805_2012Metric" (at 44.958 34.29 90)
       (effects (font (size 1.27 1.27)) hide)
     )
@@
       (effects (font (size 1.27 1.27)))
     )
-    (property "Footprint" "Resistor_SMD:R_0603_1608Metric" (at 72.39 49.022 90)
-      (effects (font (size 1.27 1.27)) hide)
-    )
+    (property "Footprint" "Resistor_SMD:R_0805_2012Metric" (at 72.39 49.022 90)
+      (effects (font (size 1.27 1.27)) hide)
+    )

Commit message: REV2
Connections:
- net GND: now also SW1.2, SW2.2, SW3.2, SW4.2
Changed lines of the file:
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@@
   (junction (at 165.1 110.49) (diameter 0) (color 0 0 0 0)
   )
+  (junction (at 165.1 49.53) (diameter 0) (color 0 0 0 0)
+  )
   (junction (at 44.45 143.51) (diameter 0) (color 0 0 0 0)
   )
@@
   (junction (at 196.85 55.88) (diameter 0) (color 0 0 0 0)
   )
+  (junction (at 165.1 36.83) (diameter 0) (color 0 0 0 0)
+  )
   (junction (at 254 63.5) (diameter 0) (color 0 0 0 0)
   )
@@
   (junction (at 165.1 53.34) (diameter 0) (color 0 0 0 0)
   )
+  (junction (at 165.1 72.39) (diameter 0) (color 0 0 0 0)
+  )
   (junction (at 96.52 111.76) (diameter 0) (color 0 0 0 0)
   )
@@
   )
   (junction (at 96.52 91.44) (diameter 0) (color 0 0 0 0)
+  )
+  (junction (at 165.1 60.96) (diameter 0) (color 0 0 0 0)
   )
   (junction (at 96.52 124.46) (diameter 0) (color 0 0 0 0)
@@
     (stroke (width 0) (type default))
   )
+  (wire (pts (xy 149.86 49.53) (xy 165.1 49.53))
+    (stroke (width 0) (type default))
+  )
   (wire (pts (xy 259.08 33.02) (xy 259.08 63.5))
     (stroke (width 0) (type default))
   )
   (wire (pts (xy 149.86 41.91) (xy 165.1 41.91))
+    (stroke (width 0) (type default))
+  )
+  (wire (pts (xy 165.1 36.83) (xy 165.1 41.91))
     (stroke (width 0) (type default))
   )
@@
     (stroke (width 0) (type default))
   )
+  (wire (pts (xy 135.89 53.34) (xy 144.78 53.34))
+    (stroke (width 0) (type default))
+  )
   (wire (pts (xy 90.17 58.42) (xy 68.58 58.42))
     (stroke (width 0) (type default))
   )
+  (wire (pts (xy 149.86 72.39) (xy 165.1 72.39))
+    (stroke (width 0) (type default))
+  )
   (wire (pts (xy 223.52 50.8) (xy 233.68 50.8))
     (stroke (width 0) (type default))
@@
     (stroke (width 0) (type default))
   )
+  (wire (pts (xy 149.86 60.96) (xy 165.1 60.96))
+    (stroke (width 0) (type default))
+  )
   (wire (pts (xy 99.06 154.94) (xy 96.52 154.94))
     (stroke (width 0) (type default))
   )
-  (wire (pts (xy 165.1 64.77) (xy 165.1 81.28))
+  (wire (pts (xy 165.1 64.77) (xy 165.1 72.39))
     (stroke (width 0) (type default))
   )
@@
     (stroke (width 0) (type default))
   )
+  (wire (pts (xy 165.1 60.96) (xy 165.1 64.77))
+    (stroke (width 0) (type default))
+  )
   (wire (pts (xy 96.52 101.6) (xy 99.06 101.6))
     (stroke (width 0) (type default))
   )
   (wire (pts (xy 156.21 110.49) (xy 165.1 110.49))
+    (stroke (width 0) (type default))
+  )
+  (wire (pts (xy 165.1 72.39) (xy 165.1 81.28))
     (stroke (width 0) (type default))
   )
@@
     (stroke (width 0) (type default))
   )
-  (wire (pts (xy 165.1 53.34) (xy 165.1 64.77))
+  (wire (pts (xy 165.1 53.34) (xy 165.1 60.96))
     (stroke (width 0) (type default))
   )
@@
     (stroke (width 0) (type dash))
   )
+  (wire (pts (xy 165.1 49.53) (xy 165.1 53.34))
+    (stroke (width 0) (type default))
+  )
   (wire (pts (xy 271.78 27.94) (xy 223.52 27.94))
     (stroke (width 0) (type default))
@@
     (stroke (width 0) (type default))
   )
-  (wire (pts (xy 165.1 29.21) (xy 165.1 41.91))
+  (wire (pts (xy 165.1 29.21) (xy 165.1 36.83))
     (stroke (width 0) (type default))
   )
@@
     (stroke (width 0) (type default))
   )
-  (wire (pts (xy 135.89 53.34) (xy 144.78 53.34))
-    (stroke (width 0) (type default))
-  )
   (wire (pts (xy 215.9 91.44) (xy 215.9 90.17))
     (stroke (width 0) (type default))
@@
     (stroke (width 0) (type default))
   )
+  (wire (pts (xy 149.86 36.83) (xy 165.1 36.83))
+    (stroke (width 0) (type default))
+  )
   (wire (pts (xy 96.52 73.66) (xy 99.06 73.66))
     (stroke (width 0) (type default))
@@
     (stroke (width 0) (type default))
   )
-  (wire (pts (xy 165.1 41.91) (xy 165.1 53.34))
-    (stroke (width 0) (type default))
-  )
+  (wire (pts (xy 165.1 41.91) (xy 165.1 49.53))
+    (stroke (width 0) (type default))
+  )
