File: hardware/kicad-project/Untitled.kicad_sch (KiCad schematic)
At the start: 37 parts, among them CN2 ST-0322D00-071-1A2H, Q1 DMG2301L-7, SW10 TS-1187A-B-A-B, SW9 TS-1187A-B-A-B, U1 ESP32-S3-WROOM-1-N8, U2 MCP73831-2ACI/MC, U3 ME6217C33P5G, U6 MAX98357AETE+T

Commit message: exports
Parts:
- removed C6: 0.1uF, Capacitor_SMD:C_0603_1608Metric, symbol Device:C
- added TP1, TP2: TestPoint, TestPoint:TestPoint_Pad_D1.0mm, symbol Connector:TestPoint
- R6: value 100k -> ???k
- R7: value 100k -> 0
Connections:
- net +3.3V: now also R7.1, TP2.1; no longer R6.1, U1.2 (3V3)
- net AMP_EN: now also U1.7 (IO7); no longer U1.8 (IO15)
- net at H2.1, U6.10 (OUTN): now also R6.2; no longer CN2.1
- net at CN2.3, CN2.4, U6.9 (OUTP): no longer CN2.2
- net GAIN_CONTROL: no longer names the net of U6.2 (GAIN_SLOT)
- net GAIN_CONTROL: no longer U1.7 (IO7)
- net JACK_DETECTION: no longer names the net of U1.10 (IO17)
- net JACK_DETECTION: no longer R7.1
- new net: R7.2, TP1.1, U1.2 (3V3)
- new net: CN2.1, R6.1
- now unconnected: CN2.6
Other:
- moved on the sheet: D1, R4

Commit message: update
Parts:
- removed U1: ESP32-S3-WROOM-1-N8, easyeda2kicad:WIFIM-SMD_ESP32-S3-WROOM-1-N8, symbol easyedaToKicad:ESP32-S3-WROOM-1-N8
- added U1: ESP32-S3-WROOM-1(N8R2), easyeda2kicad:WIRELM-SMD_ESP32-S3-WROOM-1, symbol easyedaToKicad:ESP32-S3-WROOM-1(N8R2)
- C1, C10, C11, C12, C14, C2, C3, C4, C5, C7, C8, C9: footprint Capacitor_SMD:C_0603_1608Metric -> Capacitor_SMD:C_0805_2012Metric
- R12, R13, R14, R15, R16, R3, R4, R5, R7: footprint Resistor_SMD:R_0603_1608Metric -> Resistor_SMD:R_0805_2012Metric
- R6: value ???k -> 15k; footprint Resistor_SMD:R_0603_1608Metric -> Resistor_SMD:R_0805_2012Metric
Connections:
- net AMP_EN: now also U1.7 (IO7)
- net BAT_CHARGING_STAT: now also U1.12 (IO8)
- net BAT_READ: now also U1.11 (IO18)
- net BOOT: now also U1.27 (IO0)
- net BTN_1: now also U1.22 (IO14)
- net BTN_2: now also U1.17 (IO9)
- net BTN_3: now also U1.18 (IO10)
- net BTN_4: now also U1.19 (IO11)
- net BTN_5: now also U1.20 (IO12)
- net BTN_6: now also U1.23 (IO21)
- net BTN_7: now also U1.24 (IO47)
- net EN: now also U1.3 (EN)
- net GND: now also U1.1 (GND), U1.40 (GND), U1.41 (GND)
- net GPIO_19: now also U1.13 (IO19)
- net GPIO_20: now also U1.14 (IO20)
- net I2S_BCLK: now also U1.5 (IO5)
- net I2S_DOUT: now also U1.6 (IO6)
- net I2S_LRCLK: now also U1.4 (IO4)
- net LCD_BL: now also U1.21 (IO13)
- net LCD_CS: now also U1.31 (IO38)
- net LCD_DC: now also U1.29 (IO36)
- net LCD_MOSI: now also U1.28 (IO35)
- net LCD_SCK: now also U1.30 (IO37)
- net SD_CLK: now also U1.34 (IO41)
- net SD_CMD: now also U1.35 (IO42)
- net SD_DAT_0: now also U1.33 (IO40)
- net SD_DAT_1: now also U1.32 (IO39)
- net SD_DAT_2: now also U1.39 (IO1)
- net SD_DAT_3: now also U1.38 (IO2)
- net at R7.2, TP1.1: now also U1.2 (3V3)
- no-connect marks 6 -> 7
Other:
- moved on the sheet: C1, C11, C2, R7, TP1, TP2

Commit message: rev2 almost there
Parts:
- added LED1: E6C1209RGBC3UDA, easyeda2kicad:LED-ARRAY-SMD_4P-L3.2-W2.7-TL-1, symbol easyedaToKicad:E6C1209RGBC3UDA
- added R10: 120, Resistor_SMD:R_0805_2012Metric, symbol Device:R
- added R8, R9: 30, Resistor_SMD:R_0805_2012Metric, symbol Device:R
- R6: value 15k -> 300
Connections:
- net +3.3V: now also LED1.2
- net LED_RGB_GREEN: now reaches U1.10 (IO17)
- net LED_RGB_GREEN: now also R9.2
- net LED_RGB_RED: now reaches U1.8 (IO15)
- net LED_RGB_RED: now also R10.2
- net LED_RGB_BLUE: now reaches U1.9 (IO16)
- net LED_RGB_BLUE: now also R8.2
- new net: LED1.1, R10.1
- new net: LED1.3, R9.1
- new net: LED1.4, R8.1
Other:
- note added: "RGB LED"
Changed lines of the file:
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@@
+    (stroke (width 0) (type default))
+  )
+  (wire (pts (xy 144.78 185.42) (xy 147.32 185.42))
     (stroke (width 0) (type default))
   )
@@
     (stroke (width 0) (type default))
   )
+  (wire (pts (xy 35.56 66.04) (xy 40.64 66.04))
+    (stroke (width 0) (type default))
+  )
   (wire (pts (xy 92.71 29.21) (xy 97.79 29.21))
     (stroke (width 0) (type default))
@@
     (stroke (width 0) (type default))
   )
+  (wire (pts (xy 144.78 180.34) (xy 147.32 180.34))
+    (stroke (width 0) (type default))
+  )
   (wire (pts (xy 60.96 91.44) (xy 60.96 95.25))
     (stroke (width 0) (type default))
@@
     (stroke (width 0) (type default))
   )
+  (wire (pts (xy 35.56 63.5) (xy 40.64 63.5))
+    (stroke (width 0) (type default))
+  )
   (wire (pts (xy 173.99 64.77) (xy 173.99 74.93))
     (stroke (width 0) (type default))
@@
     (stroke (width 0) (type default))
   )
+  (wire (pts (xy 137.16 166.37) (xy 137.16 170.18))
+    (stroke (width 0) (type default))
+  )
   (wire (pts (xy 90.17 171.45) (xy 90.17 173.99))
     (stroke (width 0) (type default))
@@
     (stroke (width 0) (type default))
   )
+  (wire (pts (xy 35.56 68.58) (xy 40.64 68.58))
+    (stroke (width 0) (type default))
+  )
   (wire (pts (xy 74.93 184.15) (xy 74.93 186.69))
     (stroke (width 0) (type default))
@@
   )
   (wire (pts (xy 74.93 187.96) (xy 81.28 187.96))
+    (stroke (width 0) (type default))
+  )
+  (wire (pts (xy 144.78 175.26) (xy 147.32 175.26))
     (stroke (width 0) (type default))
   )
@@
     (fill (type none))
   )
+  (rectangle (start 109.22 157.48) (end 167.64 195.58)
+    (stroke (width 0) (type dash))
+    (fill (type none))
+  )
   (text "Forbidden GPIOS : 0 3 19 20 45 46 26-37" (at 16.51 24.13 0)
     (effects (font (size 1.27 1.27)) (justify left bottom))
@@
   )
   (text "USB & Voltage protection" (at 119.38 96.52 0)
+    (effects (font (size 1.27 1.27)) (justify left bottom))
+  )
+  (text "RGB LED\n" (at 156.21 160.02 0)
     (effects (font (size 1.27 1.27)) (justify left bottom))
   )
@@
     )
   )
+  (global_label "LED_RGB_GREEN" (shape input) (at 147.32 180.34 0) (fields_autoplaced)
+    (effects (font (size 1.27 1.27)) (justify left))
+    (property "Intersheetrefs" "${INTERSHEET_REFS}" (at 165.666 180.34 0)
+      (effects (font (size 1.27 1.27)) (justify left) hide)
+    )
+  )
+  (global_label "LED_RGB_RED" (shape input) (at 35.56 63.5 180) (fields_autoplaced)
+    (effects (font (size 1.27 1.27)) (justify right))
+    (property "Intersheetrefs" "${INTERSHEET_REFS}" (at 19.6935 63.5 0)
+      (effects (font (size 1.27 1.27)) (justify right) hide)
+    )
+  )
+  (global_label "LED_RGB_BLUE" (shape input) (at 147.32 175.26 0) (fields_autoplaced)
+    (effects (font (size 1.27 1.27)) (justify left))
+    (property "Intersheetrefs" "${INTERSHEET_REFS}" (at 164.2751 175.26 0)
+      (effects (font (size 1.27 1.27)) (justify left) hide)
+    )
+  )
   (global_label "SD_CMD" (shape input) (at 87.63 58.42 0) (fields_autoplaced)
     (effects (font (size 1.27 1.27)) (justify left))
@@
     )
   )
+  (global_label "LED_RGB_RED" (shape input) (at 147.32 185.42 0) (fields_autoplaced)
+    (effects (font (size 1.27 1.27)) (justify left))
+    (property "Intersheetrefs" "${INTERSHEET_REFS}" (at 163.1865 185.42 0)
+      (effects (font (size 1.27 1.27)) (justify left) hide)
+    )
+  )
   (global_label "AMP_EN" (shape input) (at 33.02 60.96 180) (fields_autoplaced)
     (effects (font (size 1.27 1.27)) (justify right))
@@
     )
   )
+  (global_label "LED_RGB_GREEN" (shape input) (at 35.56 68.58 180) (fields_autoplaced)
+    (effects (font (size 1.27 1.27)) (justify right))
+    (property "Intersheetrefs" "${INTERSHEET_REFS}" (at 17.214 68.58 0)
+      (effects (font (size 1.27 1.27)) (justify right) hide)
+    )
+  )
   (global_label "BTN_3" (shape input) (at 55.88 95.25 270) (fields_autoplaced)
     (effects (font (size 1.27 1.27)) (justify right))
@@
     )
   )
+  (global_label "LED_RGB_BLUE" (shape input) (at 35.56 66.04 180) (fields_autoplaced)
+    (effects (font (size 1.27 1.27)) (justify right))
+    (property "Intersheetrefs" "${INTERSHEET_REFS}" (at 18.6049 66.04 0)
+      (effects (font (size 1.27 1.27)) (justify right) hide)
+    )
+  )
   (global_label "GPIO_19" (shape input) (at 33.02 76.2 180) (fields_autoplaced)
     (effects (font (size 1.27 1.27)) (justify right))
@@
         (path "/0de5ae84-7f75-4a5a-83a1-35d27fd1d8d2"
           (reference "H1") (unit 1)
+        )
+      )
+    )
+  )
+  (symbol (lib_id "easyedaToKicad:E6C1209RGBC3UDA") (at 132.08 180.34 90) (unit 1)
+    (in_bom yes) (on_board yes) (dnp no)
+    (property "Reference" "LED1" (at 130.81 165.1 90)
+      (effects (font (size 1.27 1.27)))
+    )
+    (property "Value" "E6C1209RGBC3UDA" (at 125.73 167.64 90)
+      (effects (font (size 1.27 1.27)))
+    )
+    (property "Footprint" "easyeda2kicad:LED-ARRAY-SMD_4P-L3.2-W2.7-TL-1" (at 144.78 180.34 0)
+      (effects (font (size 1.27 1.27)) hide)
+    )
+    (property "Datasheet" "https://lcsc.com/product-detail/Light-Emitting-Diodes-LED_EKINGLUX-E6C1209RGBC3UDA_C375572.html" (at 147.32 180.34 0)
+      (effects (font (size 1.27 1.27)) hide)
+    )
+    (property "LCSC Part" "C375572" (at 149.86 180.34 0)
+      (effects (font (size 1.27 1.27)) hide)
+    )
+    (pin "1")
+    (pin "2")
+    (pin "3")
+    (pin "4")
+    (instances
+      (project "Untitled"
+        (path "/0de5ae84-7f75-4a5a-83a1-35d27fd1d8d2"
+          (reference "LED1") (unit 1)
         )
       )
@@
       (effects (font (size 1.27 1.27)))
     )
-    (property "Value" "15k" (at 214.63 69.85 90)
+    (property "Value" "300" (at 214.63 69.85 90)
       (effects (font (size 1.27 1.27)))
     )
@@
     )
   )
+  (symbol (lib_id "Device:R") (at 140.97 180.34 90) (unit 1)
+    (in_bom yes) (on_board yes) (dnp no)
+    (property "Reference" "R9" (at 142.24 177.8 90)
+      (effects (font (size 1.27 1.27)) (justify left))
+    )
+    (property "Value" "30" (at 146.05 177.8 90)
+      (effects (font (size 1.27 1.27)) (justify left))
+    )
+    (property "Footprint" "Resistor_SMD:R_0805_2012Metric" (at 140.97 182.118 90)
+      (effects (font (size 1.27 1.27)) hide)
+    )
+    (property "Datasheet" "~" (at 140.97 180.34 0)
+      (effects (font (size 1.27 1.27)) hide)
+    )
+    (pin "1")
+    (pin "2")
+    (instances
+      (project "Untitled"
+        (path "/0de5ae84-7f75-4a5a-83a1-35d27fd1d8d2"
+          (reference "R9") (unit 1)
+        )
+      )
+    )
+  )
+  (symbol (lib_id "power:+3.3V") (at 137.16 166.37 0) (unit 1)
+    (in_bom yes) (on_board yes) (dnp no) (fields_autoplaced)
+    (property "Reference" "#PWR026" (at 137.16 170.18 0)
+      (effects (font (size 1.27 1.27)) hide)
+    )
+    (property "Value" "+3.3V" (at 137.16 161.29 0)
+      (effects (font (size 1.27 1.27)))
+    )
+    (property "Footprint" "" (at 137.16 166.37 0)
+      (effects (font (size 1.27 1.27)) hide)
+    )
+    (property "Datasheet" "" (at 137.16 166.37 0)
+      (effects (font (size 1.27 1.27)) hide)
+    )
+    (pin "1")
+    (instances
+      (project "Untitled"
+        (path "/0de5ae84-7f75-4a5a-83a1-35d27fd1d8d2"
+          (reference "#PWR026") (unit 1)
+        )
+      )
+    )
+  )
   (symbol (lib_id "power:GND") (at 34.29 92.71 0) (unit 1)
     (in_bom yes) (on_board yes) (dnp no) (fields_autoplaced)
@@
         (path "/0de5ae84-7f75-4a5a-83a1-35d27fd1d8d2"
           (reference "#PWR050") (unit 1)
+        )
+      )
+    )
+  )
+  (symbol (lib_id "Device:R") (at 140.97 185.42 90) (unit 1)
+    (in_bom yes) (on_board yes) (dnp no)
+    (property "Reference" "R10" (at 142.24 182.88 90)
+      (effects (font (size 1.27 1.27)) (justify left))
+    )
+    (property "Value" "120" (at 147.32 182.88 90)
+      (effects (font (size 1.27 1.27)) (justify left))
+    )
+    (property "Footprint" "Resistor_SMD:R_0805_2012Metric" (at 140.97 187.198 90)
+      (effects (font (size 1.27 1.27)) hide)
+    )
+    (property "Datasheet" "~" (at 140.97 185.42 0)
+      (effects (font (size 1.27 1.27)) hide)
+    )
+    (pin "1")
+    (pin "2")
+    (instances
+      (project "Untitled"
+        (path "/0de5ae84-7f75-4a5a-83a1-35d27fd1d8d2"
+          (reference "R10") (unit 1)
         )
       )
@@
         )
       )
+    )
+  )
+  (symbol (lib_id "Device:R") (at 140.97 175.26 90) (unit 1)
+    (in_bom yes) (on_board yes) (dnp no)
+    (property "Reference" "R8" (at 142.24 172.72 90)
+      (effects (font (size 1.27 1.27)) (justify left))
+    )
+    (property "Value" "30" (at 146.05 172.72 90)
+      (effects (font (size 1.27 1.27)) (justify left))
+    )
+    (property "Footprint" "Resistor_SMD:R_0805_2012Metric" (at 140.97 177.038 90)
+      (effects (font (size 1.27 1.27)) hide)
+    )
+    (property "Datasheet" "~" (at 140.97 175.26 0)
+      (effects (font (size 1.27 1.27)) hide)
+    )
+    (pin "1")
+    (pin "2")
+    (instances
+      (project "Untitled"
+        (path "/0de5ae84-7f75-4a5a-83a1-35d27fd1d8d2"
+          (reference "R8") (unit 1)
+        )
+      )

Commit message: REV2
Parts:
- removed TP1, TP2: TestPoint, TestPoint:TestPoint_Pad_D1.0mm, symbol Connector:TestPoint
- added R18, R19: 0, Resistor_SMD:R_0805_2012Metric, symbol Device:R
- R6: value 300 -> 330
Connections:
- net +3.3V: now also U1.2 (3V3); no longer U3.5 (VOUT)
- net +BATT: now also R19.1; no longer H1.1
- net BOOT: now also SW10.2 (B)
- net EN: now also SW9.2 (B)
- net GND: now also H1.4, H1.5, H2.4, H2.5, SW10.4 (D), SW9.4 (D), R18.2
- net at R7.2: now also U3.5 (VOUT); no longer U1.2 (3V3)
- net at U6.2 (GAIN_SLOT): now also R18.1
- new net: H1.1, R19.2
- no-connect marks 7 -> 3
Other:
- moved on the sheet: C7, C8, H1

Commit message: rev2
Parts:
- removed D3: USBLC6-2SC6, easyeda2kicad:SOT-23-6_L2.9-W1.6-P0.95-LS2.8-BL, symbol easyedaToKicad:USBLC6-2SC6
- added D2: USBLC6-2SC6_C2687116, easyeda2kicad:SOT-23-6_L2.9-W1.6-P0.95-LS2.8-BL, symbol easyedaToKicad:USBLC6-2SC6_C2687116
Connections:
- net +5V: now also D2.5 (VBUS)
- net GND: now also D2.2 (GND)
- net GPIO_19: now also D2.6 (I/O1)
- net GPIO_20: now also D2.4 (I/O2)
- net at USB1.5 (DN2), USB1.7 (DN1): now also D2.1 (I/O1)
- net at USB1.6 (DP1), USB1.8 (DP2): now also D2.3 (I/O2)
Changed lines of the file:
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@@
   (junction (at 104.14 152.4) (diameter 0) (color 0 0 0 0)
   )
+  (junction (at 166.37 123.19) (diameter 0) (color 0 0 0 0)
+  )
   (junction (at 44.45 171.45) (diameter 0) (color 0 0 0 0)
   )
@@
   (junction (at 104.14 45.72) (diameter 0) (color 0 0 0 0)
   )
-  (junction (at 166.37 128.27) (diameter 0) (color 0 0 0 0)
-  )
   (no_connect (at 50.8 91.44))
   (no_connect (at 48.26 91.44))
@@
     (stroke (width 0) (type default))
   )
-  (wire (pts (xy 166.37 129.54) (xy 170.18 129.54))
-    (stroke (width 0) (type default))
-  )
   (wire (pts (xy 63.5 91.44) (xy 63.5 95.25))
     (stroke (width 0) (type default))
@@
     (stroke (width 0) (type default))
   )
-  (wire (pts (xy 205.74 121.92) (xy 203.2 121.92))
-    (stroke (width 0) (type default))
-  )
   (wire (pts (xy 227.33 64.77) (xy 227.33 80.01))
     (stroke (width 0) (type default))
@@
     (stroke (width 0) (type default))
   )
+  (wire (pts (xy 168.91 116.84) (xy 168.91 144.78))
+    (stroke (width 0) (type default))
+  )
   (wire (pts (xy 158.75 125.73) (xy 158.75 120.65))
     (stroke (width 0) (type default))
   )
+  (wire (pts (xy 193.04 119.38) (xy 203.2 119.38))
+    (stroke (width 0) (type default))
+  )
   (wire (pts (xy 36.83 179.07) (xy 36.83 193.04))
     (stroke (width 0) (type default))
@@
     (stroke (width 0) (type default))
   )
+  (wire (pts (xy 170.18 116.84) (xy 168.91 116.84))
+    (stroke (width 0) (type default))
+  )
   (wire (pts (xy 97.79 29.21) (xy 102.87 29.21))
     (stroke (width 0) (type default))
@@
     (stroke (width 0) (type default))
   )
+  (wire (pts (xy 198.12 107.95) (xy 198.12 116.84))
+    (stroke (width 0) (type default))
+  )
   (wire (pts (xy 149.86 102.87) (xy 149.86 113.03))
     (stroke (width 0) (type default))
@@
     (stroke (width 0) (type default))
   )
+  (wire (pts (xy 193.04 114.3) (xy 203.2 114.3))
+    (stroke (width 0) (type default))
+  )
   (wire (pts (xy 233.68 125.73) (xy 234.95 125.73))
     (stroke (width 0) (type default))
@@
     (stroke (width 0) (type default))
   )
+  (wire (pts (xy 170.18 119.38) (xy 166.37 119.38))
+    (stroke (width 0) (type default))
+  )
   (wire (pts (xy 149.86 135.89) (xy 149.86 113.03))
     (stroke (width 0) (type default))
@@
     (stroke (width 0) (type default))
   )
-  (wire (pts (xy 166.37 128.27) (xy 166.37 129.54))
-    (stroke (width 0) (type default))
-  )
   (wire (pts (xy 87.63 60.96) (xy 83.82 60.96))
     (stroke (width 0) (type default))
@@
     (stroke (width 0) (type default))
   )
+  (wire (pts (xy 193.04 116.84) (xy 198.12 116.84))
+    (stroke (width 0) (type default))
+  )
   (wire (pts (xy 68.58 91.44) (xy 68.58 95.25))
     (stroke (width 0) (type default))
@@
     (stroke (width 0) (type default))
   )
+  (wire (pts (xy 166.37 119.38) (xy 166.37 123.19))
+    (stroke (width 0) (type default))
+  )
   (wire (pts (xy 92.71 124.46) (xy 92.71 147.32))
     (stroke (width 0) (type default))
@@
     )
   )
-  (global_label "GPIO_20" (shape input) (at 203.2 129.54 0) (fields_autoplaced)
+  (global_label "GPIO_20" (shape input) (at 203.2 119.38 0) (fields_autoplaced)
     (effects (font (size 1.27 1.27)) (justify left))
-    (property "Intersheetrefs" "${INTERSHEET_REFS}" (at 214.0471 129.54 0)
+    (property "Intersheetrefs" "${INTERSHEET_REFS}" (at 214.0471 119.38 0)
       (effects (font (size 1.27 1.27)) (justify left) hide)
     )
@@
     )
   )
-  (symbol (lib_id "power:+5V") (at 205.74 121.92 0) (unit 1)
+  (symbol (lib_id "power:+5V") (at 198.12 107.95 0) (unit 1)
     (in_bom yes) (on_board yes) (dnp no)
-    (property "Reference" "#PWR033" (at 205.74 125.73 0)
+    (property "Reference" "#PWR033" (at 198.12 111.76 0)
       (effects (font (size 1.27 1.27)) hide)
     )
-    (property "Value" "+5V" (at 205.74 118.11 0)
+    (property "Value" "+5V" (at 198.12 104.14 0)
       (effects (font (size 1.27 1.27)))
     )
-    (property "Footprint" "" (at 205.74 121.92 0)
+    (property "Footprint" "" (at 198.12 107.95 0)
       (effects (font (size 1.27 1.27)) hide)
     )
-    (property "Datasheet" "" (at 205.74 121.92 0)
+    (property "Datasheet" "" (at 198.12 107.95 0)
       (effects (font (size 1.27 1.27)) hide)
     )
@@
     )
   )
-  (symbol (lib_id "easyedaToKicad:USBLC6-2SC6") (at 186.69 121.92 0) (unit 1)
-    (in_bom yes) (on_board yes) (dnp no) (fields_autoplaced)
-    (property "Reference" "D3" (at 186.69 104.14 0)
-      (effects (font (size 1.27 1.27)))
-    )
-    (property "Value" "USBLC6-2SC6" (at 186.69 106.68 0)
-      (effects (font (size 1.27 1.27)))
-    )
-    (property "Footprint" "easyeda2kicad:SOT-23-6_L2.9-W1.6-P0.95-LS2.8-BL" (at 186.69 137.16 0)
-      (effects (font (size 1.27 1.27)) hide)
-    )
-    (property "Datasheet" "https://lcsc.com/product-detail/Diodes-ESD_STMicroelectronics_USBLC6-2SC6_USBLC6-2SC6_C7519.html" (at 186.69 139.7 0)
-      (effects (font (size 1.27 1.27)) hide)
-    )
-    (property "LCSC Part" "C7519" (at 186.69 142.24 0)
-      (effects (font (size 1.27 1.27)) hide)
-    )
-    (pin "1")
-    (pin "2")
-    (pin "3")
-    (pin "4")
-    (pin "5")
-    (pin "6")
-    (instances
-      (project "Untitled"
-        (path "/0de5ae84-7f75-4a5a-83a1-35d27fd1d8d2"
-          (reference "D3") (unit 1)
-        )
-      )
-    )
-  )
   (symbol (lib_id "Device:C") (at 97.79 25.4 180) (unit 1)
     (in_bom yes) (on_board yes) (dnp no)
@@
     )
   )
+  (symbol (lib_id "easyedaToKicad:USBLC6-2SC6_C2687116") (at 181.61 116.84 0) (unit 1)
+    (in_bom yes) (on_board yes) (dnp no) (fields_autoplaced)
+    (property "Reference" "D2" (at 181.61 106.68 0)
+      (effects (font (size 1.27 1.27)))
+    )
+    (property "Value" "USBLC6-2SC6_C2687116" (at 181.61 109.22 0)
+      (effects (font (size 1.27 1.27)))
+    )
+    (property "Footprint" "easyeda2kicad:SOT-23-6_L2.9-W1.6-P0.95-LS2.8-BL" (at 181.61 127 0)
+      (effects (font (size 1.27 1.27)) hide)
+    )
+    (property "Datasheet" "" (at 181.61 116.84 0)
+      (effects (font (size 1.27 1.27)) hide)
+    )
+    (property "LCSC Part" "C2687116" (at 181.61 129.54 0)
+      (effects (font (size 1.27 1.27)) hide)
+    )
+    (pin "1")
+    (pin "2")
+    (pin "3")
+    (pin "4")
+    (pin "5")
+    (pin "6")
+    (instances
+      (project "Untitled"
+        (path "/0de5ae84-7f75-4a5a-83a1-35d27fd1d8d2"
+          (reference "D2") (unit 1)
+        )
+      )
+    )
+  )
   (symbol (lib_id "Device:C") (at 252.73 111.76 0) (unit 1)
     (in_bom yes) (on_board yes) (dnp no)
@@
     )
   )
-  (symbol (lib_id "power:GND") (at 170.18 121.92 0) (unit 1)
+  (symbol (lib_id "power:GND") (at 168.91 144.78 0) (unit 1)
     (in_bom yes) (on_board yes) (dnp no) (fields_autoplaced)
-    (property "Reference" "#PWR038" (at 170.18 128.27 0)
+    (property "Reference" "#PWR038" (at 168.91 151.13 0)
       (effects (font (size 1.27 1.27)) hide)
     )
-    (property "Value" "GND" (at 170.18 127 0)
+    (property "Value" "GND" (at 168.91 149.86 0)
       (effects (font (size 1.27 1.27)))
     )
-    (property "Footprint" "" (at 170.18 121.92 0)
+    (property "Footprint" "" (at 168.91 144.78 0)
       (effects (font (size 1.27 1.27)) hide)
     )
-    (property "Datasheet" "" (at 170.18 121.92 0)
+    (property "Datasheet" "" (at 168.91 144.78 0)
       (effects (font (size 1.27 1.27)) hide)
     )
